File: gecko_qfn24_board/gecko_qfn24_board.sch (KiCad schematic (older format))
At the start: 9 parts, among them P1 CONN_01X09, P2 CONN_01X09, P3 USB_B, U1 EFM32HG309

Commit message: fixed printf
Parts:
- added D1: LED, LEDs:LED_0805, symbol LED
- added R3: R_Small, Resistors_SMD:R_0805, symbol R_Small
- added SW1: RST, Buttons_Switches_SMD:SW_SPST_B3U-1000P, symbol SW_SPST
- P3: symbol USB_B -> USB_B-RESCUE-gecko_qfn24_board
- renumbered C2 to C1, C3 to C2, C1 to C3, R2 to R1, R1 to R2
Connections:
- net +5V: now also P2.2 (P2); no longer P1.1 (P1)
- net GND: now also P1.1 (P1), R3.1, SW1.2 (B); no longer P2.2 (P2)
- net PA0: now reaches P1.8 (P8), U1.1 (PA0)
- net PA0: now also D1.2 (A)
- net PB13: now reaches P2.4 (P4), U1.10 (PB13)
- net PB14: now reaches P2.3 (P3), U1.11 (PB14)
- net PF0: now reaches P1.3 (P3), U1.19 (PF0)
- net PF1: now reaches P1.4 (P4), U1.20 (PF1)
- net PF2: now reaches P1.5 (P5), U1.21 (PF2)
- net PE12: now reaches P1.6 (P6), U1.23 (PE12)
- net PE13: now reaches P1.7 (P7), U1.24 (PE13)
- net PC0: now reaches P1.9 (P9), U1.3 (PC0)
- net PC1: now reaches P2.9 (P9), U1.4 (PC1)
- net PB7: now reaches P2.8 (P8), U1.5 (PB7)
- net PB8: now reaches P2.7 (P7), U1.6 (PB8)
- net RST: now reaches P2.6 (P6), U1.7 (~RESET)
- net RST: now also SW1.1 (A)
- net PB11: now reaches P2.5 (P5), U1.8 (PB11)
- new net: D1.1 (K), R3.2
